File: romeo-pcb.kicad_pcb (KiCad board)
At the start: 2 copper layers, 247.7 x 99.2 mm, 125 parts, among them J1 AVR-ISP-6, SW0 KEYSW, SW1 KEYSW, SW10 KEYSW, SW11 KEYSW, SW12 KEYSW, SW13 KEYSW, SW14 KEYSW, SW15 KEYSW, SW16 KEYSW, SW17 KEYSW, SW18 KEYSW, SW19 KEYSW, SW2 KEYSW, SW20 KEYSW, SW21 KEYSW, SW22 KEYSW, SW23 KEYSW, SW24 KEYSW, SW25 KEYSW, SW26 KEYSW, SW27 KEYSW, SW28 KEYSW, SW29 KEYSW, SW3 KEYSW, SW30 KEYSW, SW31 KEYSW, SW32 KEYSW, SW33 KEYSW, SW34 KEYSW, SW35 KEYSW, SW36 KEYSW, SW37 KEYSW, SW38 KEYSW, SW39 KEYSW, SW4 KEYSW, SW40 KEYSW, SW41 KEYSW, SW42 KEYSW, SW43 KEYSW, SW44 KEYSW, SW45 KEYSW, SW5 KEYSW, SW6 KEYSW, SW7 KEYSW, SW8 KEYSW, SW9 KEYSW, U1 ATmega328P-PU, Y1 Crystal

Commit message: Update romeo-pcb.kicad_pcb
Parts:
- moved G*** 31.5 mm to (176.1, 101.8) (x2)
- moved SW23 31.5 mm to (47.6, 108.7)
- moved SW24 31.5 mm to (78.6, 108.7)
- moved SW26 31.5 mm to (116.7, 108.7)
- moved SW29 31.5 mm to (173.8, 108.7)
- moved SW31 31.5 mm to (211.9, 108.7)
- moved SW33 31.5 mm to (257.2, 108.7)
- moved SW34 31.5 mm to (38.1, 127.8)
- moved SW35 31.5 mm to (59.5, 127.8)
- moved SW36 31.5 mm to (78.6, 127.8)
- moved SW37 31.5 mm to (81.0, 127.8)
- moved SW38 31.5 mm to (114.3, 127.8)
- moved SW44 31.5 mm to (261.9, 127.8)
- moved J1 31.5 mm to (121.7, 47.5)
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Other:
- board size 247.7 x 99.2 mm -> 247.6 x 99.2 mm

Commit message: Update romeo-pcb.kicad_pcb
Parts:
- added D47: D_Small, cftkb:D_DO-35_SOD27_P5.08mm_Horizontal, F.Cu at (53.3, 53.7)
- added G***: LOGO, logos:rev1_16mm_mask, B.Cu at (115.0, 136.9)
- added G***: LOGO, logos:coseyfannitutti_16mm, F.Cu at (176.0, 118.1)
- added G***: LOGO, logos:rev1_copper, B.Cu at (115.0, 136.9)
- added G***: LOGO, logos:coseyfannitutti_16mm, B.Cu at (127.3, 131.5)
- added G***: LOGO, logos:coseyfannitutti_rev1_16mm_copper, B.Cu at (127.3, 131.5)
- added G***: LOGO, logos:ROMEO_20MM_MASK, B.Cu at (161.8, 133.0)
- added G***: LOGO, logos:ROMEO_20MM_COPPER, B.Cu at (161.8, 133.0)
- added G***: LOGO, logos:rev1_copper, F.Cu at (188.3, 123.5)
- added G***: LOGO, logos:rev1_16mm_mask, F.Cu at (188.3, 123.5)
- added G***: LOGO, logos:coseyfannitutti_rev1_16mm_copper, F.Cu at (176.0, 118.1)
- added SW46: KEYSW, cftkb:SW_Cherry_MX1A_1.25u_PCBNOSCREEN, F.Cu at (38.1, 108.7)
- added SW47: KEYSW, cftkb:SW_Cherry_MX1A_1.00u_PCB-NOSCREEN, F.Cu at (59.5, 108.7)
- moved D7 3.38 mm to (141.3, 53.7)
- moved D14 3.38 mm to (73.6, 53.7)
- moved D18 3.38 mm to (124.3, 53.7)
- moved D20 3.38 mm to (131.1, 53.7)
- moved D27 3.38 mm to (93.9, 53.7)
- moved D3 3.38 mm to (80.4, 53.7)
- moved D30 3.38 mm to (117.6, 53.7)
- moved D38 3.38 mm to (87.1, 53.7)
- moved D4 3.38 mm to (100.7, 53.7)
- moved D41 3.38 mm to (107.4, 53.7)
- moved D1 3.38 mm to (56.7, 53.7)
- moved D13 3.38 mm to (60.1, 53.7)
- moved D24 3.38 mm to (66.8, 53.7)
- moved D36 3.38 mm to (63.4, 53.7)
- moved D15 3.38 mm to (83.7, 53.7)
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Routing:
- net Net-(D47-Pad2): track 0.00 -> 63.3 mm
- net Net-(D23-Pad2): track 53.7 -> 63.2 mm
- net col0: track 229.8 -> 236.6 mm
- net Net-(D6-Pad2): track 36.9 -> 40.9 mm
- net Net-(D7-Pad2): track 58.2 -> 61.9 mm
- net Net-(D3-Pad2): track 50.6 -> 47.2 mm
- net Net-(D4-Pad2): track 25.5 -> 22.1 mm
- net Net-(D16-Pad2): track 53.0 -> 49.6 mm
- net Net-(D38-Pad2): track 92.2 -> 88.8 mm
- net Net-(D26-Pad2): track 71.2 -> 67.8 mm
- net Net-(D15-Pad2): track 62.5 -> 59.2 mm
- net Net-(D27-Pad2): track 86.8 -> 83.4 mm
- net Net-(D36-Pad2): track 83.9 -> 80.8 mm
- net Net-(D13-Pad2): track 50.7 -> 47.6 mm
- net Net-(D24-Pad2): track 59.4 -> 56.4 mm
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Other:
- board text added: "SPLIT"
- board text removed: "coseyfannitutti 2019 rev1"
