File: romeo-pcb.sch (KiCad schematic (older format))
At the start: 111 parts, among them J1 AVR-ISP-6, SW0 KEYSW, SW1 KEYSW, SW10 KEYSW, SW11 KEYSW, SW12 KEYSW, SW13 KEYSW, SW14 KEYSW, SW15 KEYSW, SW16 KEYSW, SW17 KEYSW, SW18 KEYSW, SW19 KEYSW, SW2 KEYSW, SW20 KEYSW, SW21 KEYSW, SW22 KEYSW, SW23 KEYSW, SW24 KEYSW, SW25 KEYSW, SW26 KEYSW, SW27 KEYSW, SW28 KEYSW, SW29 KEYSW, SW3 KEYSW, SW30 KEYSW, SW31 KEYSW, SW32 KEYSW, SW33 KEYSW, SW34 KEYSW, SW35 KEYSW, SW36 KEYSW, SW37 KEYSW, SW38 KEYSW, SW39 KEYSW, SW4 KEYSW, SW40 KEYSW, SW41 KEYSW, SW42 KEYSW, SW43 KEYSW, SW44 KEYSW, SW45 KEYSW, SW5 KEYSW, SW6 KEYSW, SW7 KEYSW, SW8 KEYSW, SW9 KEYSW, U1 ATmega328P-PU, Y1 Crystal

Commit message: Update romeo-pcb.sch
Parts:
- added D47: D_Small, cftkb:D_DO-35_SOD27_P5.08mm_Horizontal, symbol Device:D_Small
- added SW46: KEYSW, cftkb:SW_Cherry_MX1A_1.25u_PCBNOSCREEN, symbol keyboard_parts:KEYSW
- added SW47: KEYSW, cftkb:SW_Cherry_MX1A_1.00u_PCB-NOSCREEN, symbol keyboard_parts:KEYSW
Connections:
- net col0: now also SW46.1
- net col1: now also SW47.1
- net row2: now also D47.1 (K)
- net at D23.2 (A), SW23.2: now also SW46.2
- new net: D47.2 (A), SW47.2
Changed lines of the file:
@@
 	9350 2950 10200 2950
 Wire Wire Line
-	900  2375 2575 2375
+	900  2375 1725 2375
 Connection ~ 2575 2375
 Wire Wire Line
@@
 Connection ~ 2325 1625
 Wire Wire Line
-	2325 1625 2325 2700
+	2325 1625 2325 2125
 Wire Wire Line
 	1500 1100 1500 1625
@@
 	-25  1625 -25  1575
 Connection ~ 900  1625
+$Comp
+L keyboard_parts:KEYSW SW46
+U 1 1 5DDA954C
+P 300 2075
+F 0 "SW46" H 300 2308 60  0000 C CNN
+F 1 "KEYSW" H 300 1975 60  0001 C CNN
+F 2 "cftkb:SW_Cherry_MX1A_1.25u_PCBNOSCREEN" H 300 2075 60  0001 C CNN
+F 3 "" H 300 2075 60  0000 C CNN
+	1    300  2075
+	1    0    0    -1
+$EndComp
+Wire Wire Line
+	600  2075 1150 2075
+Wire Wire Line
+	1150 2075 1150 2125
+Wire Wire Line
+	1150 2125 1500 2125
+Wire Wire Line
+	0    2075 0    2125
+Wire Wire Line
+	0    2125 900  2125
+Connection ~ 900  2125
+$Comp
+L keyboard_parts:KEYSW SW47
+U 1 1 5DDEC3B1
+P 2025 2125
+F 0 "SW47" H 2025 2358 60  0000 C CNN
+F 1 "KEYSW" H 2025 2025 60  0001 C CNN
+F 2 "cftkb:SW_Cherry_MX1A_1.00u_PCB-NOSCREEN" H 2025 2125 60  0001 C CNN
+F 3 "" H 2025 2125 60  0000 C CNN
+	1    2025 2125
+	1    0    0    -1
+$EndComp
+Connection ~ 2325 2125
+Wire Wire Line
+	2325 2125 2325 2700
+$Comp
+L Device:D_Small D47
+U 1 1 5DDEE842
+P 1725 2275
+F 0 "D47" V 1771 2207 50  0000 R CNN
+F 1 "D_Small" V 1680 2207 50  0000 R CNN
+F 2 "cftkb:D_DO-35_SOD27_P5.08mm_Horizontal" V 1725 2275 50  0001 C CNN
+F 3 "~" V 1725 2275 50  0001 C CNN
+	1    1725 2275
+	0    -1   -1   0
+$EndComp
+Connection ~ 1725 2375
+Wire Wire Line
+	1725 2375 2575 2375
+Wire Wire Line
+	1725 2125 1725 2175
 $EndSCHEMATC

Commit message: Update romeo-pcb.sch
Parts:
- BOOT1, RESET1: symbol keyboard_parts:SW_PUSH -> romeo-pcb-rescue:SW_PUSH-keyboard_parts
- F1: value 100mA -> 500mA
- J1: symbol Connector:AVR-ISP-6 -> romeo-pcb-rescue:AVR-ISP-6-Connector
- U1: symbol MCU_Microchip_ATmega:ATmega328P-PU -> romeo-pcb-rescue:ATmega328P-PU-MCU_Microchip_ATmega
Changed lines of the file:
@@
 EESchema Schematic File Version 4
-LIBS:romeo-pcb-cache
 EELAYER 30 0
 EELAYER END
@@
 $EndDescr
 $Comp
-L MCU_Microchip_ATmega:ATmega328P-PU U1
+L romeo-pcb-rescue:ATmega328P-PU-MCU_Microchip_ATmega U1
 U 1 1 5D2C1379
 P 2500 5425
@@
 P 8000 4025
 F 0 "F1" H 8068 4071 50  0000 L CNN
-F 1 "100mA" H 8068 3980 50  0000 L CNN
+F 1 "500mA" H 8068 3980 50  0000 L CNN
 F 2 "cftkb:polyfuse_5.1mm" H 8050 3825 50  0001 L CNN
 F 3 "~" H 8000 4025 50  0001 C CNN
@@
 reset
 $Comp
-L keyboard_parts:SW_PUSH RESET1
+L romeo-pcb-rescue:SW_PUSH-keyboard_parts RESET1
 U 1 1 5D2FCD08
 P 4275 4300
@@
 	5700 4425 5700 4575
 $Comp
-L keyboard_parts:SW_PUSH BOOT1
+L romeo-pcb-rescue:SW_PUSH-keyboard_parts BOOT1
 U 1 1 5D2C0447
 P 4275 4950
@@
 sck
 $Comp
-L Connector:AVR-ISP-6 J1
+L romeo-pcb-rescue:AVR-ISP-6-Connector J1
 U 1 1 5D2C325D
 P 5750 6250
